File: KiCad/esp32-vehicle-board/esp32-vehicle-board.kicad_sch (KiCad schematic)
At the start: 0 parts

Commit message: Completed Schematic
Parts:
- added C10, C11, C7: 10uF, symbol Device:C_Small
- added C12, C8, C9: 0.1uF, symbol Device:C_Small
- added D5: RED LED, symbol Device:LED
- added J1: USB_C_Receptacle_USB2.0_14P, symbol Connector:USB_C_Receptacle_USB2.0_14P
- added R1, R2: 5.1k, symbol Device:R
- added R3: 5.1k, symbol Device:R_Small
- added R4: 0, symbol Device:R_Small
- added U1: ESP32-S3-WROOM-1, RF_Module:ESP32-S3-WROOM-1, symbol RF_Module:ESP32-S3-WROOM-1
- added U3: SGM2212-3.3XKC3G, easyeda2kicad:SOT-223-3_L6.5-W3.4-P2.30-LS7.0-BR, symbol easyeda2kicad:SGM2212-3.3XKC3G_TR_C3294699
Connections:
- new net: J1.A5 (CC1), R1.1
- new net: J1.B5 (CC2), R2.1
- new net: D5.2 (A), R3.2
- new net CHIP_PU: U1.3 (EN)
- new net ESP_3V3: R4.2, U1.2 (3V3)
- new net GND: C10.2, C11.2, C12.2, C7.1, C8.1, C9.2, D5.1 (K), J1.A1 (GND), J1.A12 (GND), J1.B1 (GND), J1.B12 (GND), R1.2, R2.2, U1.1 (GND), U1.40 (GND), U1.41 (GND), U3.1 (GND)
- new net GPIO0: U1.27 (IO0)
- new net GPIO1: U1.39 (IO1)
- new net GPIO10: U1.18 (IO10)
- new net GPIO11: U1.19 (IO11)
- new net GPIO12: U1.20 (IO12)
- new net GPIO13: U1.21 (IO13)
- new net GPIO14: U1.22 (IO14)
- new net GPIO15: U1.8 (IO15)
- new net GPIO16: U1.9 (IO16)
- new net GPIO17: U1.10 (IO17)
- new net GPIO18: U1.11 (IO18)
- new net GPIO19: U1.23 (IO21)
- new net GPIO2: U1.38 (IO2)
- new net GPIO3: U1.15 (IO3)
- new net GPIO35: U1.28 (IO35)
- new net GPIO36: U1.29 (IO36)
- new net GPIO37: U1.30 (IO37)
- new net GPIO38: U1.31 (IO38)
- new net GPIO39: U1.32 (IO39)
- new net GPIO4: U1.4 (IO4)
- new net GPIO40: U1.33 (IO40)
- new net GPIO41: U1.34 (IO41)
- new net GPIO42: U1.35 (IO42)
- new net GPIO45: U1.26 (IO45)
- new net GPIO46: U1.16 (IO46)
- new net GPIO5: U1.5 (IO5)
- new net GPIO6: U1.6 (IO6)
- new net GPIO7: U1.7 (IO7)
- new net GPIO8: U1.12 (IO8)
- new net GPIO9: U1.17 (IO9)
- new net U0RXD: U1.36 (RXD0)
- new net U0TXD: U1.37 (TXD0)
- new net USB_D+: J1.A6 (D+), J1.B6 (D+), U1.14 (USB_D+)
- new net USB_D-: J1.A7 (D-), J1.B7 (D-), U1.13 (USB_D-)
- new net VCC_3V3: C10.1, C11.1, C12.1, C9.1, R3.1, R4.1, U3.2 (VOUT), U3.4 (VOUT)
- new net VCC_5V: C7.2, C8.2, J1.A4 (VBUS), J1.A9 (VBUS), J1.B4 (VBUS), J1.B9 (VBUS), U3.3 (VIN)
- no-connect marks 0 -> 2
