File: KiCad/esp32-breadboard-board/esp32-breadboard-board.kicad_pcb (KiCad board)
At the start: 2 copper layers, 21 x 72 mm, 23 parts, among them J2 Conn_01x22_Pin, J3 Conn_01x22_Pin, SW1 BOOT, SW2 EN, U1 ESP32-S3-WROOM-1, U2 USBLC6-2SC6, U3 SGM2212-3.3XKC3G

Commit message: Updated Journal and PCB
Parts:
- removed R4: 0, Resistor_SMD:R_0603_1608Metric
- added D1: D_Schottky_Small, easyeda2kicad:SOD-123_L2.7-W1.6-LS3.7-RD, F.Cu at (163.5, 105.5)
- C11, C12: moved to B.Cu
- F1: footprint Fuse:Fuse_1206_3216Metric -> Fuse:Fuse_0402_1005Metric
- R1, R2, R3, R5, R6: footprint Resistor_SMD:R_0603_1608Metric -> Resistor_SMD:R_0402_1005Metric
- moved C12 63.3 mm to (154.5, 53.5)
- moved C11 56.4 mm to (155.1, 52.3)
- moved R6 53.3 mm to (157.5, 73.0)
- moved D5 43.2 mm to (164.0, 91.6), turned to -90 degrees
- moved R3 42.3 mm to (164.3, 94.1), turned to 90 degrees
- moved R5 41.3 mm to (165.0, 108.0), turned to 90 degrees
- moved R2 40.2 mm to (163.0, 113.4), turned to 90 degrees
- moved C10 40.1 mm to (164.0, 96.5), turned to 90 degrees
- moved SW1 37.1 mm to (165.5, 111.8), turned to 90 degrees
- moved R1 36.5 mm to (158.5, 113.4), turned to 90 degrees
- moved C7 34.7 mm to (157.0, 104.5), turned to 90 degrees
- moved C9 26.7 mm to (165.2, 97.1), turned to 90 degrees
- moved SW2 26.5 mm to (155.5, 112.0), turned to 90 degrees
- moved C14 15.6 mm to (156.5, 108.0), turned to -90 degrees
- moved C8 10.7 mm to (158.2, 103.9), turned to 90 degrees
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Connections:
- C10 pad 1: VCC_3V3 -> ESP_3V3
- C11 pad 1: VCC_3V3 -> ESP_3V3
- C12 pad 1: VCC_3V3 -> ESP_3V3
- C9 pad 1: VCC_3V3 -> ESP_3V3
- F1 pad 2: VCC_5V -> Net-(D1-A)
- J3 pad 1: GND -> GPIO45
- J3 pad 10: GPIO37 -> GPIO38
- J3 pad 11: GPIO38 -> GPIO39
- J3 pad 12: GPIO39 -> GPIO40
- J3 pad 13: GPIO40 -> GPIO41
- J3 pad 14: GPIO41 -> GPIO42
- J3 pad 15: GPIO42 -> U0RXD
- J3 pad 16: U0RXD -> U0TXD
- J3 pad 17: U0TXD -> GPIO2
- J3 pad 18: GPIO2 -> GPIO1
- J3 pad 19: GPIO1 -> VCC_5V
- J3 pad 2: GPIO45 -> GPIO48
- J3 pad 20: VCC_5V -> GND
- J3 pad 3: GPIO48 -> GPIO47
- J3 pad 4: GPIO47 -> GPIO21
- J3 pad 5: GPIO21 -> GPIO14
- J3 pad 6: GPIO14 -> GPIO13
- J3 pad 7: GPIO13 -> GPIO35
- J3 pad 8: GPIO35 -> GPIO36
- J3 pad 9: GPIO36 -> GPIO37
- R3 pad 1: VCC_3V3 -> ESP_3V3
- U3 pad 2: VCC_3V3 -> ESP_3V3
- U3 pad 4: VCC_3V3 -> ESP_3V3
Routing:
- net ESP_3V3: track 0.00 -> 97.9 mm, vias 0 -> 2
- net GPIO1: track 0.00 -> 67.3 mm, vias 0 -> 1
- net /CHIP_PU: track 0.00 -> 67.0 mm, vias 0 -> 5
- net GPIO2: track 0.00 -> 63.8 mm, vias 0 -> 1
- net U0TXD: track 0.00 -> 59.0 mm, vias 0 -> 1
- net GPIO4: track 0.00 -> 58.8 mm, vias 0 -> 1
- net U0RXD: track 0.00 -> 54.9 mm, vias 0 -> 1
- net GPIO5: track 0.00 -> 54.9 mm, vias 0 -> 1
- net D-: track 0.00 -> 54.1 mm, vias 0 -> 2
- net D+: track 0.00 -> 52.6 mm, vias 0 -> 4
- net GPIO0: track 0.00 -> 52.0 mm, vias 0 -> 2
- net GPIO42: track 0.00 -> 50.7 mm, vias 0 -> 1
- net GPIO6: track 0.00 -> 50.5 mm, vias 0 -> 1
- net GPIO41: track 0.00 -> 46.6 mm, vias 0 -> 1
- net GPIO7: track 0.00 -> 46.4 mm, vias 0 -> 1
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- added copper zone on B.Cu, net GND
- added copper zone on F.Cu, net GND
Other:
- board size 21 x 72 mm -> 21 x 73 mm
