File: KiCad/esp32-breadboard-board/esp32-breadboard-board.kicad_pcb (KiCad board)
At the start: 2 copper layers, 21 x 73 mm, 23 parts, among them J2 Conn_01x22_Pin, J3 Conn_01x22_Pin, SW1 BOOT, SW2 EN, U1 ESP32-S3-WROOM-1, U2 USBLC6-2SC6, U3 SGM2212-3.3XKC3G

Commit message: commit
Parts:
- added C13: 10uF, Capacitor_SMD:C_0603_1608Metric, F.Cu at (157.7, 111.0)
- added C15: 0.1uF, Capacitor_SMD:C_0402_1005Metric, F.Cu at (159.0, 108.5)
Connections:
- USBC1 pad GND: unconnected-(USBC1-EH-Pad2) -> (no net)
Routing:
- net VBUS: track 19.8 -> 26.0 mm
Other:
- board text added: "3V3"
- board text added: "ESP32 HERE"
- board text added: "GND"
- board text added: "IO1"
- board text added: "IO10"
- board text added: "IO11"
- board text added: "IO12"
- board text added: "IO13"
- board text added: "IO14"
- board text added: "IO15"
- board text added: "IO16"
- board text added: "IO17"
- board text added: "IO18"
- board text added: "IO2"
- board text added: "IO21"
- board text added: "IO3"
- board text added: "IO35"
- board text added: "IO36"
- board text added: "IO37"
- board text added: "IO38"
- board text added: "IO39"
- board text added: "IO4"
- board text added: "IO40"
- board text added: "IO41"
- board text added: "IO42"
- board text added: "IO45"
- board text added: "IO46"
- board text added: "IO47"
- board text added: "IO48"
- board text added: "IO5"
- board text added: "IO6"
- board text added: "IO7"
- board text added: "IO8"
- board text added: "IO9"
- board text added: "RESET"
- board text added: "RX"
- board text added: "TX"
- board text added: "VCC"
- board text added: "VOIDLESS_PSYCHO"

Commit message: Updated BOM
Parts:
- removed U3: SGM2212-3.3XKC3G, easyeda2kicad:SOT-223-3_L6.5-W3.4-P2.30-LS7.0-BR
- added U4: AMS1117-3.3, Package_TO_SOT_SMD:SOT-223-3_TabPin2, F.Cu at (160.8, 100.0)
- moved D5 1.59 mm to (164.0, 90.1)
- moved C10 1.59 mm to (164.0, 94.9)
- moved C9 1.59 mm to (165.2, 95.5)
- moved R3 1.59 mm to (164.2, 92.5)
- moved C7 0.72 mm to (157.0, 105.2)
- moved C8 0.71 mm to (158.2, 104.6)
- moved R1 0.12 mm to (158.5, 113.5)
Routing:
- net ESP_3V3: track 97.9 -> 84.5 mm
- net D+: track 52.6 -> 50.7 mm, vias 4 -> 2
- net Net-(D5-A): track 0.88 -> 0.00 mm
- net GND: track 34.0 -> 34.2 mm, vias 18 -> 17
